Commit message: Added collision and visual meshes for kuka

File: resources/kuka_iiwa/kuka_iiwa.urdf (robot description, URDF)
Before this commit: robot kuka_iiwa, 8 links, 7 joints
Links:
- link link6: geometry visual mesh filename=hand.obj scale=1 1 1; visual mesh filename=meshes/link6.obj scale=1 1 1

Commit message: Stable one arm manipulation demo 4

File: resources/kuka_iiwa/kuka_iiwa.urdf (robot description, URDF)
Before this commit: robot kuka_iiwa, 8 links, 7 joints
Links:
- link link6: geometry visual mesh filename=hand2.obj scale=1 1 1; visual mesh filename=meshes/link6.obj scale=1 1 1
